Commit message: Snapshot uncommitted work before pushing to SoudruhuRobot hub
Co-Authored-By: Claude Opus 5.5 <noreply@anthropic.com>

File: ros2_ws/src/hwr_description/urdf/hwr.urdf (robot description, URDF)
Before this commit: robot hwr_rosorin_pro, 18 links, 17 joints
Links:
- added link depth_camera_link
Joints:
- added joint depth_camera_alias_joint: type fixed, parent depth_cam_frame, child depth_camera_link, origin xyz=0 0 0 rpy=0 0 0
- joint depth_cam_joint: origin xyz=0 0 0 rpy=-1.5707963267948966 0 -1.5707963267948966 -> xyz=0 0 0 rpy=1.5707963267948966 0 -1.5707963267948966
